File: PCB/Hackpad+.kicad_pcb (KiCad board)
At the start: 2 copper layers, 57.4 x 81 mm, 29 parts, among them SW1 RotaryEncoder_Switch, SW10 SW_Push, SW13 SW_Push, SW14 SW_Push, SW15 SW_Push, SW16 SW_Push, SW17 SW_Push, SW18 SW_Push, SW4 SW_Push, SW7 SW_Push, U1 XIAO-RP2040-DIP

Commit message: changed files
Parts:
- added D18: 1N4148, Diode_THT:D_DO-35_SOD27_P7.62mm_Horizontal, F.Cu at (139.4, 58.4)
Connections:
- SW1 pad A: Net-(U1-GPIO2/SCK) -> a
- SW1 pad B: Net-(U1-GPIO1/RX) -> b
- SW1 pad C: GND -> unconnected-(SW1-PadC)
- SW1 pad S1: Net-(U1-GPIO4/MISO) -> Net-(D18-A)
- SW1 pad S2: GND -> COL1
- U1 pad 10: Net-(U1-GPIO4/MISO) -> a
- U1 pad 11: unconnected-(U1-GPIO3/MOSI-Pad11) -> ROW0
- U1 pad 8: Net-(U1-GPIO1/RX) -> unconnected-(U1-GPIO1/RX-Pad8)
- U1 pad 9: Net-(U1-GPIO2/SCK) -> b
Routing:
- net COL1: track 66.2 -> 110.8 mm
- net Net-(U1-GPIO4/MISO): track 44.6 -> 0.00 mm
- net GND: track 241.7 -> 205.0 mm, vias 4 -> 6
- net Net-(D18-A): track 0.00 -> 24.3 mm
- net a: track 0.00 -> 24.0 mm
- net Net-(U1-GPIO2/SCK): track 23.4 -> 0.00 mm
- net Net-(U1-GPIO1/RX): track 22.4 -> 0.00 mm
- net b: track 0.00 -> 22.0 mm
- net Net-(D1-DOUT): track 29.8 -> 48.2 mm, vias 0 -> 2
- net Net-(D3-DIN): track 44.7 -> 32.1 mm
- net ROW0: track 0.00 -> 9.86 mm
- net Net-(D14-DOUT): track 31.3 -> 25.0 mm
- net +5V: track 204.6 -> 198.7 mm, vias 4 -> 7
- net Net-(D24-A): track 14.4 -> 10.7 mm, vias 1 -> 0
- net DIN: track 41.9 -> 38.5 mm, vias 0 -> 1
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